File: PingPong_388_2019 rev2.brd (EAGLE design)
At the start: 53 x 50.8 mm, 21 parts, among them IC1 7805T, U2 ATMEGA328PB-AUR

Commit message: Add files via upload
Parts:
- added U$1, U$2: (no value), holes:3,0
- moved IC1 3.59 mm to (68.6, 35.6)
- moved C6 2.84 mm to (35.6, 33.0)
- moved BARELL_JACK 2.54 mm to (48.3, 44.5)
- moved D2 1.80 mm to (40.6, 33.0)
- moved LED2 1.27 mm to (53.3, 11.4)
Routing:
- net GND: track 213.2 -> 220.8 mm
- net CRYSTAL2: track 11.6 -> 15.6 mm
- net 12V: track 25.6 -> 24.0 mm
- net N$3: track 2.99 -> 4.26 mm
- net RESET: track 27.5 -> 28.6 mm
- net 5V: track 143.4 -> 142.8 mm
Other:
- outline, holes or cut-outs redrawn
